File: 01_MT7981_DDR4.kicad_sch (KiCad schematic)
At the start: 116 parts, among them U1 MT7981B_BGA

Commit message: Update to Kicad format 9
Parts:
- renumbered CD4 to CD?, CD24 to CD?, CD27 to CD?, CD26 to CD?, CD5 to CD?, CD21 to CD?, CD18 to CD?, CD14 to CD?, CD8 to CD?, CD19 to CD?, CD13 to CD?, CD29 to CD?, CD33 to CD?, CD25 to CD?, CD1 to CD?, CD35 to CD?, CD6 to CD?, CD28 to CD?, CD9 to CD?, CD30 to CD?, CD15 to CD?, CD22 to CD?, CD11 to CD?, CD20 to CD?, CD10 to CD?, CD12 to CD?, CD7 to CD?, CD32 to CD?, CD36 to CD?, CD37 to CD?, CD31 to CD?, CD17 to CD?, CD34 to CD?, CD2 to CD?, CD3 to CD?, CD16 to CD?, CD23 to CD?, CP8 to CP?, CP5 to CP?, CP2 to CP?, CP4 to CP?, CP10 to CP?, CP3 to CP?, CP6 to CP?, CP11 to CP?, CP1 to CP?, CP7 to CP?, CP9 to CP?, L1 to L?, RD11 to RD?, RD6 to RD?, RD10 to RD?, RD13 to RD?, RD9 to RD?, RD15 to RD?, RD1 to RD?, RD7 to RD?, RD2 to RD?, RD8 to RD?, RD12 to RD?, RD3 to RD?, RD5 to RD?, RD4 to RD?, RD14 to RD?, RP4 to RP?, RP6 to RP?, RP2 to RP?, RP9 to RP?, RP3 to RP?, RP11 to RP?, RP8 to RP?, RP1 to RP?, RP5 to RP?, RP10 to RP?, RP7 to RP?, TP1 to TP?, TP2 to TP?, TP3 to TP?, TPD18 to TPD?, TPD11 to TPD?, TPD28 to TPD?, TPD21 to TPD?, TPD19 to TPD?, TPD9 to TPD?, TPD3 to TPD?, TPD10 to TPD?, TPD17 to TPD?, TPD32 to TPD?, TPD31 to TPD?, TPD14 to TPD?, TPD20 to TPD?, TPD2 to TPD?, TPD6 to TPD?, TPD13 to TPD?, TPD7 to TPD?, TPD22 to TPD?, TPD4 to TPD?, TPD23 to TPD?, TPD15 to TPD?, TPD16 to TPD?, TPD27 to TPD?, TPD24 to TPD?, TPD26 to TPD?, TPD8 to TPD?, TPD1 to TPD?, TPD25 to TPD?, TPD30 to TPD?, TPD12 to TPD?, TPD29 to TPD?, TPD5 to TPD?, U1 to U?, * to U?, UD1 to UD?, UP3 to UP?, UP2 to UP?, UP1 to UP?
Connections:
- net AVDD18_EMI0: no longer U?.R17 (AVDD18_RDDR)
- net AVDDQ_EMI0: no longer U?.M11 (VDDIO_DDR_R), U?.M12 (VDDIO_DDR_CA), U?.N10 (VDDIO_DDR_MCLK), U?.N8 (VDDIO_DDR_DQ), U?.N9 (VDDIO_DDR_DQ)
- net DVDD08: no longer U?.L11 (DVDD_DDR_TX), U?.L12 (DVDD_DDR_RX)
- net EMI0_A0: no longer U?.T14 (EMI0_A0/EMI0_A0)
- net EMI0_A1: no longer U?.U12 (EMI0_A1/EMI0_A1)
- net EMI0_A10: no longer U?.R16 (EMI0_A10/EMI0_BA2)
- net EMI0_A11: no longer U?.T15 (EMI0_A11/EMI0_A9)
- net EMI0_A12: no longer U?.R13 (EMI0_A12/EMI0_A10)
- net EMI0_A13: no longer U?.T12 (EMI0_A13/EMI0_A8)
- net EMI0_A2: no longer U?.U16 (EMI0_A2/EMI0_A13)
- net EMI0_A3: no longer U?.U13 (EMI0_A3/EMI0_A14)
- net EMI0_A4: no longer U?.R14 (EMI0_A4/EMI0_CAS_N)
- net EMI0_A5: no longer U?.T11 (EMI0_A5/EMI0_A4)
- net EMI0_A6: no longer U?.V17 (EMI0_A6/EMI0_A7)
- net EMI0_A7: no longer U?.V13 (EMI0_A7/EMI0_A6)
- net EMI0_A8: no longer U?.T16 (EMI0_A8/EMI0_A3)
- net EMI0_A9: no longer U?.T13 (EMI0_A9/EMI0_A11)
- net EMI0_ACT_N: no longer U?.V18 (EMI0_ACT_N/EMI0_BA0)
- net EMI0_BA0: no longer U?.U17 (EMI0_BA0/EMI0_A5)
- net EMI0_BA1: no longer U?.R11 (EMI0_BA1/EMI0_BA1)
- net EMI0_BG0: no longer U?.V16 (EMI0_BG0/EMI0_A2)
- net EMI0_CAS_N: no longer U?.V14 (EMI0_CAS_N/EMI0_A12)
- net EMI0_CKE0: no longer U?.U11 (EMI0_CKE0/EMI0_CKE0)
- net EMI0_CK_C: no longer U?.V11 (EMI0_CK_C/EMI0_CK_C)
- net EMI0_CK_T: no longer U?.U10 (EMI0_CK_T/EMI0_CK_T)
- net EMI0_CS0_N_1: no longer U?.V19 (EMI0_CS0_N/EMI0_CS0_N)
- net EMI0_DM0: now also U?.D9 (AVSS18_WBG); no longer U?.U7 (EMI0_DM0/EMI0_DM0)
- net EMI0_DM1: now also U?.E10 (AVSS18_WBG); no longer U?.T5 (EMI0_DM1/EMI0_DM1)
- net EMI0_DQ0: no longer U?.U5 (EMI0_DQ0/EMI0_DQ0)
- net EMI0_DQ1: now also U?.E11 (AVDD12_WBG); no longer U?.V8 (EMI0_DQ1/EMI0_DQ1)
- net EMI0_DQ10: now also U?.C16 (AVSS18_WBG); no longer U?.T7 (EMI0_DQ10/EMI0_DQ9)
- net EMI0_DQ11: now also U?.C6 (AVSS18_WBG); no longer U?.R9 (EMI0_DQ11/EMI0_DQ14)
- net EMI0_DQ12: now also U?.B15 (AVSS18_WBG); no longer U?.T6 (EMI0_DQ12/EMI0_DQ13)
- net EMI0_DQ13: now also U?.B6 (AVSS18_WBG); no longer U?.R10 (EMI0_DQ13/EMI0_DQ10)
- net EMI0_DQ14: now also U?.A14 (AVSS18_WBG); no longer U?.R6 (EMI0_DQ14/EMI0_DQ11)
- net EMI0_DQ15: now also U?.A7 (AVSS18_WBG); no longer U?.T9 (EMI0_DQ15/EMI0_DQ8)
- net EMI0_DQ2: now also U?.E12 (AVDD18_WBG); no longer U?.V5 (EMI0_DQ2/EMI0_DQ2)
- net EMI0_DQ3: no longer U?.U8 (EMI0_DQ3/EMI0_DQ3)
- net EMI0_DQ4: no longer U?.U4 (EMI0_DQ4/EMI0_DQ6)
- net EMI0_DQ5: now also U?.D12 (AVSS18_WBG); no longer U?.U9 (EMI0_DQ5/EMI0_DQ7)
- net EMI0_DQ6: now also U?.D13 (AVSS18_WBG); no longer U?.V4 (EMI0_DQ6/EMI0_DQ4)
- net EMI0_DQ7: now also U?.D10 (AVSS18_WBG); no longer U?.V10 (EMI0_DQ7/EMI0_DQ5)
- net EMI0_DQ8: now also U?.D11 (AVSS18_WBG); no longer U?.R7 (EMI0_DQ8/EMI0_DQ15)
- net EMI0_DQ9: now also U?.A11 (AVSS18_WBG); no longer U?.T10 (EMI0_DQ9/EMI0_DQ12)
- net EMI0_DQS0_C: now also U?.E9 (AVSS18_WBG); no longer U?.V7 (EMI0_DQS0_C/EMI0_DQS0_C)
- net EMI0_DQS0_T: no longer U?.U6 (EMI0_DQS0_T/EMI0_DQS0_T)
- net EMI0_DQS1_C: no longer U?.T8 (EMI0_DQS1_C/EMI0_DQS1_C)
- net EMI0_DQS1_T: no longer U?.R8 (EMI0_DQS1_T/EMI0_DQS1_T)
- net EMI0_ODT: no longer U?.U15 (EMI0_ODT/EMI0_ODT)
- net EMI0_RAS_N: no longer U?.U14 (EMI0_RAS_N/EMI0_RAS_N)
- net EMI0_WE_N: no longer U?.U18 (EMI0_WE_N/EMI0_WE_N)
- net EMI_EXTR: no longer U?.U19 (EMI_EXTR)
- net EMI_RESET_N: no longer U?.R15 (EMI_RESET_N)
