File: 02_MT7981_Power_AFE.kicad_sch (KiCad schematic)
At the start: 84 parts, among them U1 MT7981B_BGA

Commit message: Update to Kicad format 9
Connections:
- net 1.8VD: no longer U1.L6 (DVDD18IO_BL)
- net 1.8VD_1: no longer U1.L16 (DVDD18IO_RB)
- net 3.3VD: no longer U1.M6 (DVDD33IO_LB)
- net AVDD12_CKSQ: no longer U1.E15 (AVDD12_CKSQ)
- net AVDD15_POR: no longer U1.A3 (AVDD15_POR)
- net AVDD18_AUXADC: no longer U1.G20 (AVDD18_AUXADC)
- net AVDD18_CKSQ: no longer U1.E14 (AVDD18_CKSQ)
- net AVDD18_PLLGP: no longer U1.J5 (AVDD18_PLLGP)
- net AVDD18_POR: no longer U1.C4 (AVDD18_POR)
- net DVDD18_VQPS: now also U1.D2 (WF_CBA_RESETB); no longer U1.E5 (DVDD18_VQPS)
- net GND: now also U1.A11 (AVSS18_WBG), U1.A14 (AVSS18_WBG), U1.A7 (AVSS18_WBG), U1.B15 (AVSS18_WBG), U1.B6 (AVSS18_WBG), U1.C1 (WF_TOP_DATA), U1.C16 (AVSS18_WBG), U1.C2 (WF_XO_REQ), U1.C6 (AVSS18_WBG), U1.D10 (AVSS18_WBG), U1.D11 (AVSS18_WBG), U1.D13 (AVSS18_WBG), U1.D14 (AVSS18_WBG), U1.D15 (AVSS18_WBG), U1.D2 (WF_CBA_RESETB), U1.D3 (WF_DIG_RESETB), U1.D8 (AVSS18_WBG), U1.D9 (AVSS18_WBG), U1.E10 (AVSS18_WBG), U1.E13 (AVSS18_WBG), U1.E3 (WF_TOP_CLK), U1.E9 (AVSS18_WBG); no longer U1.D17 (GNDK), U1.D4 (GNDK), U1.E1 (GNDK), U1.E16 (GNDK), U1.E17 (GNDK), U1.E2 (GNDK), U1.E4 (GNDK), U1.F11 (GNDK), U1.F12 (GNDK), U1.F18 (GNDK), U1.F3 (GNDK), U1.F5 (GNDK), U1.G10 (GNDK), U1.G11 (GNDK), U1.G12 (GNDK), U1.G18 (GNDK), U1.G3 (GNDK), U1.G5 (GNDK), U1.G8 (GNDK), U1.G9 (GNDK), U1.H1 (GNDK), U1.H10 (GNDK), U1.H11 (GNDK), U1.H12 (GNDK), U1.H13 (GNDK), U1.H16 (GNDK), U1.H17 (GNDK), U1.H18 (GNDK), U1.H4 (GNDK), U1.H5 (GNDK), U1.H7 (GNDK), U1.H8 (GNDK), U1.H9 (GNDK), U1.J10 (GNDK), U1.J11 (GNDK), U1.J12 (GNDK), U1.J13 (GNDK), U1.J14 (GNDK), U1.J16 (GNDK), U1.J17 (GNDK), U1.J2 (GNDK), U1.J3 (GNDK), U1.J7 (GNDK), U1.J8 (GNDK), U1.J9 (GNDK), U1.K10 (GNDK), U1.K11 (GNDK), U1.K12 (GNDK), U1.K13 (GNDK), U1.K15 (GNDK), U1.K16 (GNDK), U1.K18 (GNDK), U1.K5 (GNDK), U1.K7 (GNDK), U1.K8 (GNDK), U1.K9 (GNDK), U1.L13 (GNDK), U1.L18 (GNDK), U1.L19 (GNDK), U1.L20 (GNDK), U1.M13 (GNDK), U1.M16 (GNDK), U1.M5 (GNDK), U1.N11 (GNDK), U1.N12 (GNDK), U1.N13 (GNDK), U1.N14 (GNDK), U1.N15 (GNDK), U1.N16 (GNDK), U1.N17 (GNDK), U1.N18 (GNDK), U1.N5 (GNDK), U1.N6 (GNDK), U1.N7 (GNDK), U1.P10 (GNDK), U1.P11 (GNDK), U1.P12 (GNDK), U1.P13 (GNDK), U1.P14 (GNDK), U1.P15 (GNDK), U1.P16 (GNDK), U1.P17 (GNDK), U1.P4 (GNDK), U1.P5 (GNDK), U1.P6 (GNDK), U1.P7 (GNDK), U1.P8 (GNDK), U1.P9 (GNDK), U1.R5 (GNDK), U1.T17 (GNDK), U1.T18 (GNDK), U1.T4 (GNDK), U1.U20 (GNDK), U1.U3 (GNDK), U1.V12 (GNDK), U1.V15 (GNDK), U1.V3 (GNDK), U1.V6 (GNDK), U1.V9 (GNDK)
- net VCCK: now also U1.A14 (AVSS18_WBG), U1.A7 (AVSS18_WBG), U1.B15 (AVSS18_WBG), U1.B6 (AVSS18_WBG), U1.C6 (AVSS18_WBG), U1.D14 (AVSS18_WBG), U1.D15 (AVSS18_WBG), U1.D8 (AVSS18_WBG), U1.D9 (AVSS18_WBG), U1.E10 (AVSS18_WBG), U1.E13 (AVSS18_WBG), U1.E9 (AVSS18_WBG); no longer U1.F10 (VCCK), U1.F13 (VCCK), U1.F14 (VCCK), U1.F8 (VCCK), U1.F9 (VCCK), U1.G13 (VCCK), U1.G6 (VCCK), U1.G7 (VCCK), U1.H14 (VCCK), U1.J6 (VCCK), U1.K14 (VCCK), U1.L10 (VCCK), U1.L14 (VCCK), U1.L8 (VCCK), U1.L9 (VCCK), U1.M14 (VCCK), U1.M15 (VCCK), U1.M7 (VCCK)
- net at TPD33.1: no longer U1.L1 (PLLGP_TP)
- net at TPD34.1: no longer U1.L2 (PLLGP_TN)
