File: 03_MT7981_PCIe_USB_GPHY.kicad_sch (KiCad schematic)
At the start: 113 parts, among them CON3 Header-1x2, Q1 MMBT3904, Q28 MMBT3904, Q42 MMBT3904, SW1 SW-CFG-DIPx1, SW2 TS-038-H7, SW3 TS-038-H7, U1 MT7981B_BGA, U16 EM6324QYSP5B-2.8+, U2 W25Q128JVSIQ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

Commit message: Update to Kicad format 9
Connections:
- net AUXIN0: no longer U1.F19 (AUXIN0)
- net AUXIN1: no longer U1.F20 (AUXIN1)
- net AUXIN2: no longer U1.E20 (AUXIN2)
- net AVDD09_PCIE: no longer U1.G4 (AVDD09_PCIE)
- net AVDD09_SGMII: no longer U1.J18 (AVDD09_SGMII)
- net AVDD18_COM: no longer U1.R18 (AVDD18_COM)
- net AVDD18_PCIE: no longer U1.F4 (AVDD18_PCIE)
- net AVDD18_SGMII: no longer U1.H19 (AVDD18_SGMII)
- net AVDD18_USB: no longer U1.J4 (AVDD18_USB)
- net AVDD33_LD_P0: no longer U1.P18 (AVDD33_LD_P0)
- net AVDD33_USB: no longer U1.K4 (AVDD33_USB)
- net ESW_P0_A_TXVn: no longer U1.R20 (GBE_TXVN_A_P0)
- net ESW_P0_A_TXVp: no longer U1.T20 (GBE_TXVP_A_P0)
- net ESW_P0_B_TXVn: no longer U1.P19 (GBE_TXVN_B_P0)
- net ESW_P0_B_TXVp: no longer U1.R19 (GBE_TXVP_B_P0)
- net ESW_P0_C_TXVn: no longer U1.N20 (GBE_TXVN_C_P0)
- net ESW_P0_C_TXVp: no longer U1.N19 (GBE_TXVP_C_P0)
- net ESW_P0_D_TXVn: no longer U1.M19 (GBE_TXVN_D_P0)
- net ESW_P0_D_TXVp: no longer U1.M20 (GBE_TXVP_D_P0)
- net GBE_LEDA: no longer U1.M2 (WF5G_LED)
- net GBE_LEDB: now also U1.E11 (AVDD12_WBG); no longer U1.M1 (WF2G_LED)
- net GND: now also U1.D2 (WF_CBA_RESETB); no longer U1.F16 (TESTMODE)
- net GPIO_RESETn: no longer U1.E18 (GPIO_RESET)
- net GPIO_WPS: no longer U1.F17 (GPIO_WPS)
- net HW_INT_8811: no longer U1.M17 (GBE_INT)
- net HW_RSTN_8811: no longer U1.M18 (GBE_RESET)
- net JTAG_JTCK: no longer U1.N4 (JTAG_JTCLK)
- net JTAG_JTDI: no longer U1.L4 (JTAG_JTDI)
- net JTAG_JTDO: no longer U1.M3 (JTAG_JTDO)
- net JTAG_JTMS: no longer U1.L5 (JTAG_JTMS)
- net JTAG_JTRST_N: no longer U1.M4 (JTAG_JTRST_N)
- net MAIN_X40M: no longer U1.D16 (MAIN_X40M_IN)
- net MT7981_BG_OUT: no longer U1.A4 (POR_BG_OUT)
- net MT7981_MD: no longer U1.E19 (TSAUX_MD)
- net MT7981_REFP: no longer U1.G19 (TSAUX_REFP)
- net MT7981_REXT: no longer U1.T19 (REXT)
- net MT7981_SYSRSTB_3P3V: now also U1.C2 (WF_XO_REQ); no longer U1.N2 (SYSRSTB)
- net PCIE_PERESETn: now also U1.E12 (AVDD18_WBG); no longer U1.N3 (PCIE_PERESET_N)
- net PMU_RSTB_1P8V: no longer U1.B4 (POR_RSTB)
- net PWM0: now also U1.E11 (AVDD12_WBG); no longer U1.D20 (PWM0)
- net SMI_MDC: no longer U1.L17 (SMI_MDC)
- net SMI_MDIO: no longer U1.K17 (SMI_MDIO)
- net SOC_HSGMII_RXn: no longer U1.J20 (SGMII_LN0_RXN)
- net SOC_HSGMII_RXp: no longer U1.J19 (SGMII_LN0_RXP)
- net SOC_HSGMII_TXn: no longer U1.K20 (SGMII_LN0_TXN)
- net SOC_HSGMII_TXp: no longer U1.K19 (SGMII_LN0_TXP)
- net SOC_PCIe_CLKn: now also U1.D14 (AVSS18_WBG); no longer U1.H3 (PCIE_CKN)
- net SOC_PCIe_CLKp: now also U1.D15 (AVSS18_WBG); no longer U1.H2 (PCIE_CKP)
- net SOC_PCIe_RXn: now also U1.D9 (AVSS18_WBG); no longer U1.G2 (PCIE_LN0_RXN)
- net SOC_PCIe_RXp: now also U1.E10 (AVSS18_WBG); no longer U1.G1 (PCIE_LN0_RXP)
- net SOC_PCIe_TXn: now also U1.E9 (AVSS18_WBG); no longer U1.F1 (PCIE_LN0_TXN)
- net SOC_PCIe_TXp: no longer U1.F2 (PCIE_LN0_TXP)
- net SOC_U2USB_DM: now also U1.B15 (AVSS18_WBG); no longer U1.K3 (USB_DM)
- net SOC_U2USB_DP: now also U1.B6 (AVSS18_WBG); no longer U1.K2 (USB_DP)
- net SPI0_CLK: now also U1.B6 (AVSS18_WBG); no longer U1.D19 (SPI0_CLK)
- net SPI0_CS: now also U1.C16 (AVSS18_WBG); no longer U1.B20 (SPI0_CS)
- net SPI0_HOLD: now also U1.A7 (AVSS18_WBG); no longer U1.B19 (SPI0_HOLD)
- net SPI0_MISO: now also U1.C6 (AVSS18_WBG); no longer U1.C18 (SPI0_MISO)
- net SPI0_MOSI: now also U1.B15 (AVSS18_WBG); no longer U1.D18 (SPI0_MOSI)
- net SPI0_WP: now also U1.A14 (AVSS18_WBG); no longer U1.C19 (SPI0_WP)
- net SPI1_CLK: now also U1.E13 (AVSS18_WBG); no longer U1.A19 (SPI1_CLK)
- net SPI1_CS: now also U1.D8 (AVSS18_WBG); no longer U1.C17 (SPI1_CS)
- net SPI1_MISO: now also U1.D9 (AVSS18_WBG); no longer U1.A18 (SPI1_MISO)
- net SPI1_MOSI: now also U1.E10 (AVSS18_WBG); no longer U1.B18 (SPI1_MOSI)
- net SPI2_CLK: no longer U1.T2 (SPI2_CLK)
- net SPI2_CS: no longer U1.V2 (SPI2_CS)
- net SPI2_HOLD: no longer U1.U2 (SPI2_HOLD)
- net SPI2_MISO: no longer U1.T1 (SPI2_MISO)
- net SPI2_MOSI: no longer U1.T3 (SPI2_MOSI)
- net SPI2_WP: no longer U1.U1 (SPI2_WP)
- net SYS_WATCHDOG_3P3V: no longer U1.R1 (SYS_WATCHDOG)
- net UART0_RXD_DEBUG: no longer U1.G16 (UART0_RXD)
- net UART0_TXD_DEBUG: no longer U1.G17 (UART0_TXD)
- net USB_VBUS: no longer U1.L3 (USB_VBUS)
- net WO_JTCK: no longer U1.P3 (WO_JTAG_JTCLK)
- net WO_JTDI: no longer U1.R4 (WO_JTAG_JTDI)
- net WO_JTDO: no longer U1.R3 (WO_JTAG_JTDO)
- net WO_JTMS: no longer U1.P2 (WO_JTAG_JTMS)
- net WO_JTRST_N: no longer U1.R2 (WO_JTAG_JTRST_N)
