File: 05_MT7976C_DBDC.kicad_sch (KiCad schematic)
At the start: 226 parts, among them U8 MT7976C, X1 40MHz,10pF,10PPM

Commit message: Update to Kicad format 9
Parts:
- renumbered ANT3 to ANT?, ANT9 to ANT?, ANT5 to ANT?, BF10 to BF?, BF12 to BF?, BF11 to BF?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
