File: 07_M2_KEYM_mikroBUS_EEPROM_RTC.kicad_sch (KiCad schematic)
At the start: 109 parts, among them CN10 M2_KEYM_42H, CN6 FTSH-105-01-L-DV-007-K, CN7 Header-SIP1x8-PH254-X2, CON2 Battery_Cell, U13 AT8563S //SPL8563M //PCF8563TS, U14 N~{C}P24C02A-TSH-MIR, X3 32.768KHz,9pF,20PPM

Commit message: Update to Kicad format 9
Parts:
- renumbered C96 to C?, C114 to C?, C95 to C?, C98 to C?, C5 to C?, C4 to C?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
